Commit message: fix: add front caster so robot no longer tips nose-down

File: src/indoor_bot_description/urdf/indoor_bot.gazebo.xacro (robot description, xacro)
@@ -25,4 +25,9 @@
   <!-- rear caster: frictionless so it doesn't drag against the diff-drive motion -->
   <gazebo reference="caster_link">
+    <mu1>0</mu1>
+    <mu2>0</mu2>
+  </gazebo>
+  <!-- front caster: frictionless so it doesn't drag against the diff-drive motion -->
+  <gazebo reference="front_caster_link">
     <mu1>0</mu1>
     <mu2>0</mu2>

File: src/indoor_bot_description/urdf/indoor_bot.urdf.xacro (robot description, xacro)
@@ -17,4 +17,5 @@
   <xacro:property name="caster_mass" value="0.05"/>
   <xacro:property name="caster_x_offset" value="-0.12"/>
+  <xacro:property name="caster_front_x_offset" value="0.12"/>
   <!-- base_footprint -> base_link: wheel-radius height above the ground -->
   <xacro:property name="base_link_z" value="${wheel_radius}"/>
@@ -112,4 +113,25 @@
     <origin xyz="${caster_x_offset} 0 ${caster_z_offset}" rpy="0 0 0"/>
   </joint>
+  <!-- front caster: stops the body tipping forward -->
+  <link name="front_caster_link">
+    <visual>
+      <geometry>
+        <sphere radius="${caster_radius}"/>
+      </geometry>
+    </visual>
+    <collision>
+      <geometry>
+        <sphere radius="${caster_radius}"/>
+      </geometry>
+    </collision>
+    <xacro:inertia_sphere mass="${caster_mass}" radius="${caster_radius}">
+      <origin xyz="0 0 0" rpy="0 0 0"/>
+    </xacro:inertia_sphere>
+  </link>
+  <joint name="front_caster_joint" type="fixed">
+    <parent link="base_link"/>
+    <child link="front_caster_link"/>
+    <origin xyz="${caster_front_x_offset} 0 ${caster_z_offset}" rpy="0 0 0"/>
+  </joint>
   <!-- ================= base_scan (2D LiDAR) ================= -->
   <link name="base_scan">
